File: _saved_Livolo_EU_2Gang_1way.sch (KiCad schematic (older format))
At the start: 39 parts, among them IC1 ATMEGA328P, U1 ATSHA204A, U2 RFM69_MINIMAL

Commit message: rootage
Connections:
- net L1_RST: now also IC1.1 (PD3(INT1)); no longer IC1.2 (PD4(XCK/T0))
- net TOUCH_1: now also IC1.2 (PD4(XCK/T0)); no longer IC1.1 (PD3(INT1))
Changed lines of the file:
@@
 Text Label 15350 3450 2    65   ~ 0
 IRQ
-Text Label 8950 3950 2    65   ~ 0
+Text Label 8950 3850 2    65   ~ 0
 L1_RST
 Text Label 11850 8550 0    65   ~ 0
 L1_RST
-Text Label 8950 3850 2    65   ~ 0
+Text Label 8950 3950 2    65   ~ 0
 TOUCH_1
 Text Label 11850 8350 0    65   ~ 0
@@
 Text Label 15050 3450 0    10   ~ 0
 IRQ
-Text Label 8450 3950 0    10   ~ 0
-L1_RST
 Text Label 11750 8550 0    10   ~ 0
 L1_RST
